File: Circuit/circuit.sch (EAGLE design)
At the start: 10 parts, among them U2 CAT24C32

Commit message: database upload
Parts:
- added J1: POWER_JACK, SparkFun-Connectors:POWER_JACK
- added JP2: (no value), adafruit:PINHD-1X8BIG
- added LED1, LED2, LED3: (no value), adafruit:LEDSQR2X5
- added R1: (no value), adafruit:R-US_0411/12
- added T1, T2: 2N2222, adafruit:2N2222
- added U$1: TSOP38238, radu-eagle-lib:TSOP38238
Connections:
- new net 12V: J1.PWR, LED2.A, LED3.A
- new net N$1: LED2.C, T1.C
- new net N$2: LED3.C, T2.C
- new net N$3: J1.GND, J1.GNDBREAK
- net GND: now also T1.E, T2.E
Changed lines of the file:
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@@
 <layer number="112" name="tSilk" color="7" fill="1" visible="yes" active="yes"/>
 <layer number="113" name="ReferenceLS" color="7" fill="1" visible="no" active="no"/>
+<layer number="114" name="Badge_Outline" color="7" fill="1" visible="yes" active="yes"/>
+<layer number="115" name="ReferenceISLANDS" color="7" fill="1" visible="yes" active="yes"/>
 <layer number="116" name="Patch_BOT" color="9" fill="4" visible="yes" active="yes"/>
 <layer number="118" name="Rect_Pads" color="7" fill="1" visible="no" active="no"/>
@@
 <part name="FID3" library="microbuilder" deviceset="FIDUCIAL" device="&quot;&quot;"/>
 <part name="FID4" library="microbuilder" deviceset="FIDUCIAL" device="&quot;&quot;"/>
+<part name="U$1" library="radu-eagle-lib" deviceset="TSOP38238" device=""/>
+<part name="R1" library="adafruit" library_urn="urn:adsk.eagle:library:420" deviceset="R-US_" device="0411/12"/>
+<part name="LED1" library="adafruit" library_urn="urn:adsk.eagle:library:420" deviceset="LED" device="SQR2X5"/>
+<part name="JP2" library="adafruit" library_urn="urn:adsk.eagle:library:420" deviceset="PINHD-1X8" device="BIG"/>
+<part name="J1" library="SparkFun-Connectors" deviceset="POWER_JACK" device=""/>
+<part name="T1" library="adafruit" library_urn="urn:adsk.eagle:library:420" deviceset="2N2222" device=""/>
+<part name="T2" library="adafruit" library_urn="urn:adsk.eagle:library:420" deviceset="2N2222" device=""/>
+<part name="LED2" library="adafruit" library_urn="urn:adsk.eagle:library:420" deviceset="LED" device="SQR2X5"/>
+<part name="LED3" library="adafruit" library_urn="urn:adsk.eagle:library:420" deviceset="LED" device="SQR2X5"/>
+<part name="GND6" library="supply1" deviceset="GND" device=""/>
+<part name="GND7" library="supply1" deviceset="GND" device=""/>
 </parts>
 <sheets>
@@
 <instance part="FID3" gate="G$1" x="45.72" y="73.66"/>
 <instance part="FID4" gate="G$1" x="20.32" y="73.66"/>
+<instance part="U$1" gate="G$1" x="81.28" y="88.9"/>
+<instance part="R1" gate="G$1" x="83.82" y="73.66"/>
+<instance part="LED1" gate="G$1" x="83.82" y="63.5"/>
+<instance part="JP2" gate="G$1" x="134.62" y="93.98"/>
+<instance part="J1" gate="G$1" x="185.42" y="93.98"/>
+<instance part="T1" gate="G$1" x="185.42" y="45.72"/>
+<instance part="T2" gate="G$1" x="213.36" y="45.72"/>
+<instance part="LED2" gate="G$1" x="187.96" y="60.96"/>
+<instance part="LED3" gate="G$1" x="215.9" y="60.96"/>
+<instance part="GND6" gate="1" x="203.2" y="30.48"/>
+<instance part="GND7" gate="1" x="195.58" y="88.9"/>
 </instances>
 <busses>
@@
 <pinref part="GND5" gate="1" pin="GND"/>
 </segment>
+<segment>
+<pinref part="T1" gate="G$1" pin="E"/>
+<pinref part="T2" gate="G$1" pin="E"/>
+<wire x1="187.96" y1="40.64" x2="203.2" y2="40.64" width="0.1524" layer="91"/>
+<pinref part="GND6" gate="1" pin="GND"/>
+<wire x1="203.2" y1="40.64" x2="215.9" y2="40.64" width="0.1524" layer="91"/>
+<wire x1="203.2" y1="33.02" x2="203.2" y2="40.64" width="0.1524" layer="91"/>
+<junction x="203.2" y="40.64"/>
+</segment>
 </net>
 <net name="VDD" class="0">
@@
 </segment>
 </net>
+<net name="12V" class="0">
+<segment>
+<pinref part="J1" gate="G$1" pin="PWR"/>
+<wire x1="187.96" y1="101.6" x2="215.9" y2="101.6" width="0.1524" layer="91"/>
+<pinref part="LED3" gate="G$1" pin="A"/>
+<wire x1="215.9" y1="101.6" x2="215.9" y2="78.74" width="0.1524" layer="91"/>
+<pinref part="LED2" gate="G$1" pin="A"/>
+<wire x1="215.9" y1="78.74" x2="215.9" y2="63.5" width="0.1524" layer="91"/>
+<wire x1="215.9" y1="78.74" x2="187.96" y2="78.74" width="0.1524" layer="91"/>
+<wire x1="187.96" y1="78.74" x2="187.96" y2="63.5" width="0.1524" layer="91"/>
+<junction x="215.9" y="78.74"/>
+</segment>
+</net>
+<net name="N$1" class="0">
+<segment>
+<pinref part="LED2" gate="G$1" pin="C"/>
+<pinref part="T1" gate="G$1" pin="C"/>
+<wire x1="187.96" y1="55.88" x2="187.96" y2="50.8" width="0.1524" layer="91"/>
+</segment>
+</net>
+<net name="N$2" class="0">
+<segment>
+<pinref part="LED3" gate="G$1" pin="C"/>
+<pinref part="T2" gate="G$1" pin="C"/>
+<wire x1="215.9" y1="55.88" x2="215.9" y2="50.8" width="0.1524" layer="91"/>
+</segment>
+</net>
+<net name="N$3" class="0">
+<segment>
+<pinref part="J1" gate="G$1" pin="GNDBREAK"/>
+<wire x1="187.96" y1="99.06" x2="195.58" y2="99.06" width="0.1524" layer="91"/>
+<wire x1="195.58" y1="99.06" x2="195.58" y2="96.52" width="0.1524" layer="91"/>
+<pinref part="J1" gate="G$1" pin="GND"/>
+<wire x1="195.58" y1="96.52" x2="195.58" y2="91.44" width="0.1524" layer="91"/>
+<wire x1="187.96" y1="96.52" x2="195.58" y2="96.52" width="0.1524" layer="91"/>
+<junction x="195.58" y="96.52"/>
+</segment>
+</net>
 </nets>
 </sheet>
@@
 </schematic>
 </drawing>
+<compatibility>
+<note version="8.2" severity="warning">
+Since Version 8.2, Eagle supports online libraries. The ids
+of those online libraries will not be understood (or retained)
+with this version.
+</note>
+</compatibility>
 </eagle>
