File: Circuit/circuit.brd (EAGLE design)
At the start: 160 x 100 mm, 19 parts, among them J1 POWER_JACK, T1 2N2222, T2 2N2222, U2 CAT24C32

Commit message: Auto stash before merge of "master" and "origin/master"
Parts:
- added B1: SPARKFUN_LOGIC_LEVEL_CONVERTER, SparkFun-Boards:SPARKFUN_LOGIC_LEVEL_CONVERTER
- added J2: RJ45, SparkFun-Connectors:RJ45-8
- added J3: 1X2-3.5MM, adafruit:1X2-3.5MM
- added T3, T4: 2N2222, adafruit:TO92-EBC-OVAL
Connections:
- removed net GPIO12: RPI1.32
- removed net GPIO16: RPI1.36
- removed net GPIO17: RPI1.11
- removed net GPIO18: RPI1.12
- removed net GPIO19: RPI1.35
- removed net GPIO21: RPI1.40
- removed net GPIO23: RPI1.16
- removed net GPIO25: RPI1.22
- removed net GPIO4: RPI1.7
- removed net GPIO5: RPI1.29
- removed net GPIO6: RPI1.31
- removed net N$1: LED2.K, T1.C
- removed net VDD: JP1.1
- new net BUT1: J2.5, RPI1.7
- new net BUT2: J2.7, RPI1.11
- new net CUE_1: B1.HV1, T1.B
- new net CUE_2: B1.HV2, T2.B
- new net CUE_BOTH: B1.HV3, T3.B, T4.B
- new net LED1: J2.2, LED3.K, T2.C, T3.C
- new net LED1_CTRL: B1.LV1, RPI1.36
- new net LED2: J2.4, LED2.K, T1.C, T4.C
- new net LED2_CTRL: B1.LV2, RPI1.31
- new net LED_BOTH_CTRL: B1.LV3, RPI1.32
- new net LIRC_IN: RPI1.16, U$1.2
- new net PWR_LED: R1.1, RPI1.29
- new net REWARD: J3.1, RPI1.22
- net 12V: now also B1.HV, J2.1, J2.3
- net 3.3V: now also B1.LV, J2.6, J2.8, U$1.3
- net 5.0V: now also JP1.1
- net BCLK: now also RPI1.12
- net DIN: now also RPI1.40
- net GND: now also B1.GND1, B1.GND2, J3.2, LED1.K, T3.E, T4.E, U$1.1
- net LRCLK: now also RPI1.35
- net N$2: now also LED1.A, R1.2; no longer LED3.K, T2.C
